Commit message: :truck: Moving files in model directory

File: src/self_balancing_robot/model/self_balancing_robot.urdf.xacro (robot description, xacro)
@@ -1,4 +1,27 @@
 <?xml version="1.0"?>
-<robot name="self_balancing_robot">
+<robot name="self_balancing_robot"
+  xmlns:xacro="http://www.ros.org/wiki/xacro">
+  <!-- Macro for color -->
+  <xacro:macro name="material_with_color" params="name color">
+    <material name="${name}">
+      <color rgba="${color}"/>
+    </material>
+  </xacro:macro>
+  <link name="dummy_root_link">
+    <visual>
+      <geometry>
+        <sphere radius="0.01"/>
+      </geometry>
+      <material name="Invisible">
+        <color rgba="0 0 0 0"/>
+      </material>
+    </visual>
+  </link>
+  <!-- Fixed Joint from Dummy Link to Base Link -->
+  <joint name="dummy_to_base_joint" type="fixed">
+    <parent link="dummy_root_link"/>
+    <child link="base_link"/>
+    <origin xyz="0 0 0" rpy="0 0 0"/>
+  </joint>
   <!-- Robot Base -->
   <link name="base_link">
@@ -9,14 +32,12 @@
     </inertial>
     <visual>
-      <origin xyz="0 0 0.1" />
+      <origin xyz="0 0 0" />
       <geometry>
         <box size="0.2 0.1 0.4" />
       </geometry>
-      <material name="Green">
-        <color rgba="0 1 0 1"/>
-      </material>
+      <xacro:material_with_color name="Green" color="0 1 0 1" />
     </visual>
     <collision>
-      <origin xyz="0 0 0.1" />
+      <origin xyz="0 0 0" />
       <geometry>
         <box size="0.2 0.1 0.4" />
@@ -35,7 +56,5 @@
         <cylinder radius="0.05" length="0.02" />
       </geometry>
-      <material name="Black">
-        <color rgba="0 0 0 1"/>
-      </material>
+      <xacro:material_with_color name="Black" color="0 0 0 1" />
     </visual>
     <collision>
@@ -56,7 +75,5 @@
         <cylinder radius="0.05" length="0.02" />
       </geometry>
-      <material name="Black">
-        <color rgba="0 0 0 1"/>
-      </material>
+      <xacro:material_with_color name="Black" color="0 0 0 1" />
     </visual>
     <collision>
@@ -66,4 +83,5 @@
     </collision>
   </link>
+  <xacro:include filename="$(find self_balancing_robot)/model/self_balancing_robot.gazebo" />
   <!-- Joint Definitions -->
   <!-- Left Wheel Joint -->
@@ -71,6 +89,8 @@
     <parent link="base_link"/>
     <child link="left_wheel"/>
-    <origin xyz="0.1 0.1 0" rpy="0 1.57 0"/>
+    <origin xyz="0.11 0.0 -0.2" rpy="0 1.57 0"/>
     <axis xyz="0 0 1"/>
+    <limit effort="5000.0" velocity="10.0"/>
+    <dynamics damping="1.0" friction="1.0"/>
   </joint>
   <!-- Right Wheel Joint -->
@@ -78,6 +98,8 @@
     <parent link="base_link"/>
     <child link="right_wheel"/>
-    <origin xyz="0.1 -0.1 0" rpy="0 1.57 0"/>
+    <origin xyz="-0.11 0.0 -0.2" rpy="0 1.57 0"/>
     <axis xyz="0 0 1"/>
+    <limit effort="5000.0" velocity="10.0"/>
+    <dynamics damping="1.0" friction="1.0"/>
   </joint>
 </robot>

Commit message: :sparkles: Integrated IMU in gazebo with ros bridge

File: src/self_balancing_robot/model/self_balancing_robot.urdf.xacro (robot description, xacro)
@@ -45,4 +45,34 @@
     </collision>
   </link>
+  <!-- IMU Sensor Link -->
+  <link name="imu_link">
+    <inertial>
+      <origin xyz="0 0 0" />
+      <mass value="0.01" />
+      <inertia ixx="1e-5" ixy="0" ixz="0" iyy="1e-5" iyz="0" izz="1e-5" />
+    </inertial>
+    <visual>
+      <origin xyz="0 0 0" />
+      <geometry>
+        <box size="0.01 0.01 0.01" />
+      </geometry>
+      <xacro:material_with_color name="Gray" color="0.5 0.5 0.5 1" />
+    </visual>
+    <collision>
+      <origin xyz="0 0 0" />
+      <geometry>
+        <box size="0.01 0.01 0.01" />
+      </geometry>
+    </collision>
+  </link>
+  <!-- Gazebo plugin for IMU -->
+  <gazebo reference="imu_link">
+    <sensor name="imu_sensor" type="imu">
+      <always_on>1</always_on>
+      <update_rate>10</update_rate>
+      <visualize>true</visualize>
+      <topic>/sensors/imu</topic>
+    </sensor>
+  </gazebo>
   <!-- Left Wheel -->
   <link name="left_wheel">
@@ -85,4 +115,11 @@
   <xacro:include filename="$(find self_balancing_robot)/model/self_balancing_robot.gazebo" />
   <!-- Joint Definitions -->
+  <!-- Joint between base_link and imu_link -->
+  <joint name="base_to_imu_joint" type="fixed">
+    <parent link="base_link"/>
+    <child link="imu_link"/>
+    <origin xyz="0 0 0.2" rpy="0 0 0"/>
+    <!-- Adjust the position as needed -->
+  </joint>
   <!-- Left Wheel Joint -->
   <joint name="left_wheel_joint" type="continuous">

Commit message: :wrench: Fixing limits

File: src/self_balancing_robot/model/self_balancing_robot.urdf.xacro (robot description, xacro)
@@ -128,5 +128,5 @@
     <origin xyz="0.11 0.0 -0.2" rpy="0 1.57 0"/>
     <axis xyz="0 0 1"/>
-    <limit effort="5000.0" velocity="10.0"/>
+    <limit effort="5000.0" velocity="500.0"/>
     <dynamics damping="1.0" friction="1.0"/>
   </joint>
@@ -137,5 +137,5 @@
     <origin xyz="-0.11 0.0 -0.2" rpy="0 1.57 0"/>
     <axis xyz="0 0 1"/>
-    <limit effort="5000.0" velocity="10.0"/>
+    <limit effort="5000.0" velocity="500.0"/>
     <dynamics damping="1.0" friction="1.0"/>
   </joint>
